File: keyboards/atari-a8/kicad/atari-keyboard.kicad_pcb (KiCad board)
At the start: 2 copper layers, 355.8 x 141.4 mm, 230 parts, among them J101 PLAYER 1, J102 PLAYER 2, J103 I2C DISPLAY, SW201 ESC, SW202 1, SW203 2, SW204 3, SW205 4, SW206 5, SW207 6, SW208 7, SW209 8, SW210 9, SW211 0, SW212 LT, SW213 GT, SW214 BS, SW215 C_UP, SW216 C_LEFT, SW217 C_DOWN, SW218 C_RIGHT, SW219 TAB, SW220 Q, SW221 W, SW222 E, SW223 R, SW224 T, SW225 Y, SW226 U, SW227 I, SW228 O, SW229 P, SW230 DASH, SW231 EQUAL, SW232 RET, SW233 HELP, SW234 RESET, SW235 OPTION, SW236 SELECT, SW237 CTRL, SW238 A, SW239 S, SW240 D, SW241 F, SW242 G, SW243 H, SW244 J, SW245 K, SW246 L, SW247 SEMI, SW248 PLUS, SW249 ASTRIX, SW250 CAPS, SW251 START, SW252 POWER, SW253 MENU, SW254 TURBO, SW255 FN, SW256 LSHIFT, SW257 Z, SW258 X, SW259 C, SW260 V, SW261 B, SW262 N, SW263 M, SW264 COMMA, SW265 PERIOD, SW266 SLASH, SW267 RSHIFT, SW268 INV, SW269 BREAK, SW270 SPACE, U101 Elite-C

Commit message: Cleaned up some more trace.
Routing:
- net C2: track 501.7 -> 495.4 mm
- net R5: track 367.0 -> 365.8 mm
- net R2: track 311.3 -> 310.5 mm
- net R4: track 306.6 -> 305.9 mm
- net R8: track 301.4 -> 300.7 mm
- net C6: track 550.4 -> 549.8 mm

Commit message: Used new standoff holes and more track cleanup work.
Parts:
- removed H201, H202, H203, H204, H205, H206, H207, H208, H209, H210, H211, H212, H213, H214, H215, H216, H217, H218, H219, H220, H221, H222, H223, H224, H225, H226, H227, H228, H229, H230, H231, H232, H233, H234, H235, H236, H237, H238, H239, H240, H241, H242, H243, H244, H245, H246, H247, H248, H249, H250, H251, H252, H253, H254, H255, H256, H257, H258, H259, H260, H261, H262, H263, H264, H265, H266, H267, H268, H269, H270: Hole, MountingHole:MountingHole_2.2mm_M2
Routing:
- net Net-(D102-Pad1): track 22.8 -> 24.5 mm
- net C8: track 409.9 -> 408.2 mm
- net Net-(D268-Pad2): track 11.3 -> 9.67 mm
- net Net-(D229-Pad2): track 11.3 -> 9.67 mm
- net Net-(D265-Pad2): track 12.2 -> 10.8 mm
- net Net-(D104-Pad1): track 24.1 -> 25.4 mm
- net C7: track 495.4 -> 494.2 mm
- net C4: track 426.7 -> 427.8 mm
- net R2: track 310.5 -> 311.1 mm
- net Net-(D246-Pad2): track 11.3 -> 10.7 mm
- net R7: track 392.0 -> 392.5 mm
- net Net-(D230-Pad2): track 12.6 -> 12.1 mm
- net Net-(D228-Pad2): track 12.6 -> 12.1 mm
- net Net-(D223-Pad2): track 11.5 -> 11.0 mm
Other:
- outline, holes or cut-outs redrawn
