File: keyboards/atari-a8/kicad/keyswitch_pcb/keyswitch_pcb.kicad_pcb (KiCad board)
At the start: 2 copper layers, 357.2 x 140.5 mm, 165 parts, among them J101 PLAYER 1, J102 Development Connector, J103 I2C DISPLAY, J104 Jumper Connector, J105 Primary Connector, SW101 RESET, SW200 ESC, SW201 1, SW202 2, SW203 3, SW204 4, SW205 5, SW206 6, SW207 7, SW208 8, SW209 TAB, SW210 Q, SW211 W, SW212 E, SW213 R, SW214 T, SW215 Y, SW216 U, SW217 I, SW218 CONTROL, SW219 A, SW220 S, SW221 D, SW222 F, SW223 G, SW224 H, SW225 J, SW226 K, SW227 LSHIFT, SW228 Z, SW229 X, SW230 C, SW231 V, SW232 B, SW233 N, SW234 M, SW235 COMMA, SW236 9, SW237 0, SW238 LT, SW239 GT, SW240 BS, SW241 BREAK, SW242 O, SW243 P, SW244 DASH, SW245 INV, SW246 C_UP, SW247 CAPS, SW248 ASTRIX, SW249 PLUS, SW250 SEMI, SW251 L, SW252 EQUAL, SW253 RETURN, SW254 SPACE, SW255 FN, SW256 PERIOD, SW257 SLASH, SW258 RSHIFT, SW259 C_LEFT, SW260 C_DOWN, SW261 C_RIGHT, SW262 SELECT, SW263 OPTION, SW264 RESET, SW265 HELP, SW266 POWER, SW267 MENU, SW268 TURBO, SW269 START, U101 MAX7219, U102 MAX7219

Commit message: Reworked mounting holes and cleaned up labeling.
Routing:
- net SW_COL2: track 0.00 -> 584.9 mm, vias 0 -> 1
- net SW_COL1: track 0.00 -> 566.1 mm, vias 0 -> 2
- net SW_ROW7: track 0.00 -> 563.9 mm
- net SW_COL3: track 0.00 -> 546.7 mm, vias 0 -> 1
- net SW_COL4: track 0.00 -> 537.3 mm, vias 0 -> 1
- net LED_COL1: track 0.00 -> 536.0 mm
- net SW_ROW8: track 0.00 -> 534.5 mm
- net SW_COL5: track 0.00 -> 511.1 mm, vias 0 -> 3
- net SW_COL6: track 0.00 -> 505.6 mm
- net SW_COL7: track 0.00 -> 502.6 mm, vias 0 -> 1
- net SW_ROW6: track 0.00 -> 502.6 mm, vias 0 -> 1
- net VCC: track 0.00 -> 490.1 mm, vias 0 -> 1
- net SW_ROW5: track 0.00 -> 477.5 mm, vias 0 -> 1
- net LED_COL2: track 0.00 -> 475.6 mm, vias 0 -> 2
- net GND: track 0.00 -> 468.8 mm
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